File: pcb/minirobot.kicad_pcb (KiCad board)
At the start: 2 copper layers, 0 parts

Commit message: more schematics
Parts:
- added C1: 0.1uF, kicadlib:CAPC2012X100N, F.Cu at (124.8, 125.2)
- added C10: 0.1uF, kicadlib:CAPC2012X100N, F.Cu at (116.4, 120.4)
- added C11: 0.1uF, kicadlib:CAPC2012X100N, F.Cu at (95.6, 135.4)
- added C12: 0.1uF, kicadlib:CAPC2012X100N, F.Cu at (104.6, 127.1)
- added C13: 0.1uF, kicadlib:CAPC2012X100N, F.Cu at (90.7, 135.4)
- added C2: 10uF, kicadlib:CAPC2012X100N, F.Cu at (97.8, 113.4)
- added C3: 1uF, kicadlib:CAPC2012X100N, F.Cu at (130.7, 120.4)
- added C4: 0.1uF, kicadlib:CAPC2012X100N, F.Cu at (214.5, 71.2)
- added C5: 10uF >6V, kicadlib:CAPC2012X100N, F.Cu at (214.0, 89.3)
- added C6: 0.1uF, kicadlib:CAPC2012X100N, F.Cu at (129.7, 125.2)
- added C7: 0.012uF, kicadlib:CAPC2012X100N, F.Cu at (213.6, 91.8)
- added C8: 10uF, kicadlib:CAPC2012X100N, F.Cu at (205.6, 102.5)
- added C9: 0.1uF, kicadlib:CAPC2012X100N, F.Cu at (100.5, 135.4)
- added D1: DIODESCH, kicadlib:SOT95P237X112_132-3N, F.Cu at (211.3, 100.4)
- added D2: ACTIVITY-BLUE, kicadlib:LEDC2012X100N, F.Cu at (92.3, 114.3)
- added D3: CONN-GREEN, kicadlib:LEDC2012X100N, F.Cu at (165.1, 131.3)
- added D4: LED, kicadlib:LEDC1608X40N, F.Cu at (235.4, 66.5)
- added D5: DIODESCH, kicadlib:SOT95P237X112_132-3N, F.Cu at (212.0, 95.3)
- added D6: 3V3LED, kicadlib:LEDC2012X100N, F.Cu at (216.5, 97.7)
- added L1: 4.7uH, kicadlib:INDC3218X180N, F.Cu at (206.3, 99.7)
- added P1: FEELERLEFT, kicadlib:OMRON-SS-5GL-F-3-RAM, F.Cu at (139.8, 44.2)
- added P2: SERVO, kicadlib:HDRV3W66P254_1X3_762X249X838P, F.Cu at (193.9, 82.0)
- added P3: BATTERY, kicadlib:HDRV2W66P254_1X2_508X249X838P, F.Cu at (205.3, 94.9)
- added P4: FEELERRIGHT, kicadlib:OMRON-SS-5GL-F-3-RA, F.Cu at (145.6, 44.8)
- added P5: SERVO, kicadlib:HDRV3W66P254_1X3_762X249X838P, F.Cu at (203.5, 77.0)
- added R1: 51R, kicadlib:RESC2012X100N, F.Cu at (219.3, 73.7)
- added R10: 0R, kicadlib:RESC2012X100N, F.Cu at (214.7, 82.0)
- added R11: 51R, kicadlib:RESC2012X100N, F.Cu at (224.2, 71.2)
- added R12: 100R, kicadlib:RESC2012X100N, F.Cu at (102.7, 113.4)
- added R13: 10K, kicadlib:RESC2012X100N, F.Cu at (221.2, 66.2)
- added R14: 100R, kicadlib:RESC2012X100N, F.Cu at (163.7, 133.8)
- added R15: 51R, kicadlib:RESC2012X100N, F.Cu at (223.1, 76.2)
- added R16: 0R, kicadlib:RESC2012X100N, F.Cu at (219.4, 71.2)
- added R17: 62K, kicadlib:RESC2012X100N, F.Cu at (218.5, 91.8)
- added R18: 20K, kicadlib:RESC2012X100N, F.Cu at (216.5, 94.3)
- added R19: 51R, kicadlib:RESC2012X100N, F.Cu at (229.4, 63.3)
- added R2: 51R, kicadlib:RESC2012X100N, F.Cu at (209.9, 82.0)
- added R20: 51R, kicadlib:RESC2012X100N, F.Cu at (226.0, 66.2)
- added R21: 100R, kicadlib:RESC2012X100N, F.Cu at (218.9, 89.3)
- added R22: 10K, kicadlib:RESC2012X100N, F.Cu at (218.3, 76.2)
- added R23: 10K, kicadlib:RESC2012X100N, F.Cu at (226.0, 68.7)
- added R24: 10K, kicadlib:RESC2012X100N, F.Cu at (229.0, 71.2)
- added R25: 0R, kicadlib:RESC2012X100N, F.Cu at (218.3, 78.7)
- added R26: 0R, kicadlib:RESC2012X100N, F.Cu at (230.8, 68.3)
- added R27: 10K, kicadlib:RESC2012X100N, F.Cu at (109.4, 129.6)
- added R28: 10K, kicadlib:RESC2012X100N, F.Cu at (116.4, 122.9)
- added R29: 4.7K, kicadlib:RESC2012X100N, F.Cu at (109.5, 127.1)
- added R3: 10K, kicadlib:RESC2012X100N, F.Cu at (229.4, 60.8)
- added R30: 4.7K, kicadlib:RESC2012X100N, F.Cu at (104.6, 129.6)
- added R4: 10K, kicadlib:RESC2012X100N, F.Cu at (234.1, 60.8)
- added R5: 10K, kicadlib:RESC2012X100N, F.Cu at (221.2, 68.7)
- added R6: 0R, kicadlib:RESC2012X100N, F.Cu at (230.8, 65.8)
- added R7: 0R, kicadlib:RESC2012X100N, F.Cu at (214.5, 73.7)
- added R8: 51R, kicadlib:RESC2012X100N, F.Cu at (234.1, 63.3)
- added R9: 10K, kicadlib:RESC2012X100N, F.Cu at (224.1, 73.7)
- added S1: POWER, kicadlib:COPAL-MFS101D-6-Z, F.Cu at (198.0, 100.4)
- added U1: LINELEFTOUT, kicadlib:QRE1113GR, F.Cu at (224.3, 61.9)
- added U10: WHEELRIGHT, kicadlib:QRE1113-RA, F.Cu at (197.0, 78.1)
- added U11: STM32SWDUART, kicadlib:HDRV8W64P254_2X4_1016X483X838P, F.Cu at (105.1, 123.3)
- added U12: STM32F411RET6, kicadlib:QFP50P1200X1200X160-64N, F.Cu at (95.7, 127.1)
- added U2: WHEELLEFT, kicadlib:QRE1113-RA, F.Cu at (216.9, 62.4)
- added U3: LINELEFTIN, kicadlib:QRE1113GR, F.Cu at (204.9, 82.0)
- added U4: TCS3472, kicadlib:TCS3472, F.Cu at (219.7, 82.4)
- added U5: RN4020, kicadlib:RN4020, F.Cu at (23.0, 146.3)
- added U6: ST-LIS3MDL, kicadlib:LGA12S50P4X4_192X192X100, F.Cu at (125.8, 121.7)
- added U7: LINERIGHTIN, kicadlib:QRE1113GR, F.Cu at (213.3, 77.6)
- added U8: DIODES-AP3211, kicadlib:SOT95P270X145-6N, F.Cu at (207.6, 91.1)
- added U9: LINERIGHTOUT, kicadlib:QRE1113GR, F.Cu at (215.9, 66.9)

Commit message: pcb routing complete
Parts:
- D4, U1, U11, U3, U4, U7, U9: moved to B.Cu
- moved U5 122.8 mm to (130.2, 86.3), turned to 270 degrees
- moved R4 121.5 mm to (112.7, 56.7), turned to 270 degrees
- moved R5 118.9 mm to (102.4, 66.7)
- moved R8 117.2 mm to (117.1, 56.7), turned to 90 degrees
- moved R6 116.2 mm to (114.9, 56.7), turned to 90 degrees
- moved U2 115.2 mm to (102.0, 70.2)
- moved R7 112.5 mm to (102.4, 64.5), turned to 180 degrees
- moved U1 111.6 mm to (113.0, 52.9)
- moved R17 111.3 mm to (107.4, 85.0), turned to 270 degrees
- moved D4 110.8 mm to (125.0, 56.0)
- moved R3 110.7 mm to (119.0, 52.3), turned to 180 degrees
- moved R1 110.1 mm to (110.5, 56.7), turned to 90 degrees
- moved R18 109.2 mm to (107.4, 88.6), turned to 270 degrees
- moved R2 107.8 mm to (102.4, 73.9), turned to 180 degrees
- moved R9 106.1 mm to (119.3, 56.7), turned to 270 degrees
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Connections:
- U12 pad 33: /Sensors/LINELEFTOUT -> /Sensors/LINERIGHTOUT
- U12 pad 34: /Sensors/LINELEFTIN -> /Sensors/LINERIGHTIN
- U12 pad 35: /Sensors/LINERIGHTOUT -> /Sensors/LINELEFTIN
- U12 pad 36: /Sensors/LINERIGHTIN -> /Sensors/LINELEFTOUT
- U12 pad 37: /Sensors/FEELERLEFT -> /Sensors/FEELERRIGHT
- U12 pad 38: /Sensors/FEELERRIGHT -> /Sensors/FEELERLEFT
Routing:
- net +3.3V: track 0.00 -> 250.0 mm, vias 0 -> 7
- net GNDPWR: track 0.00 -> 93.9 mm, vias 0 -> 33
- net /Compass/I2CSCL: track 0.00 -> 62.4 mm, vias 0 -> 6
- net /Sensors/SERVORIGHT: track 0.00 -> 50.0 mm, vias 0 -> 4
- net /Compass/I2CSDA: track 0.00 -> 49.2 mm, vias 0 -> 3
- net /Sensors/SERVOLEFT: track 0.00 -> 46.1 mm, vias 0 -> 4
- net /Sensors/WHEELLEFT: track 0.00 -> 38.1 mm, vias 0 -> 6
- net /Bluetooth/BLECONN: track 0.00 -> 37.5 mm, vias 0 -> 2
- net /DEBUGTX: track 0.00 -> 35.4 mm
- net /Bluetooth/BLEWS: track 0.00 -> 34.1 mm, vias 0 -> 2
- net /Bluetooth/BLEMLDPEV: track 0.00 -> 31.2 mm, vias 0 -> 2
- net /VBAT: track 0.00 -> 30.8 mm, vias 0 -> 2
- net Vcc: track 0.00 -> 30.1 mm
- net /DEBUGGPIO: track 0.00 -> 29.1 mm, vias 0 -> 1
- net /DEBUGRX: track 0.00 -> 29.0 mm
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- added copper zone on B.Cu, net GNDPWR
- added copper zone on F.Cu, net GNDPWR
Other:
- board outline added: 50 x 50 mm
- net class Default: clearance 0.2 -> 0.2032; trace_width 0.25 -> 0.2032; via_dia 0.6 -> 0.7366; via_drill 0.4 -> 0.381
- rule trace_clearance: 0.2 -> 0.2032
- rule trace_min: 0.2 -> 0.1524
- rule via_min_drill: 0.3 -> 0.3302
- rule via_min_size: 0.4 -> 0.6858
- board text added: "ACTIVITY"
- board text added: "CONNECTION"
- board text added: "POWER"
