File: pcb/minirobot.kicad_pcb (KiCad board)
At the start: 2 copper layers, 50 x 50 mm, 68 parts, among them P1 FEELERLEFT, P2 SERVO, P3 BATTERY, P4 FEELERRIGHT, P5 SERVO, U1 LINELEFTOUT, U10 WHEELRIGHT, U11 STM32SWDUART, U12 STM32F411RET6, U2 WHEELLEFT, U3 LINELEFTIN, U4 TCS3472, U5 RN4020, U6 ST-LIS3MDL, U7 LINERIGHTIN, U8 DIODES-AP3211, U9 LINERIGHTOUT

Commit message: 2016-02-23 pcb
Other:
- rule pad_to_mask_clearance: 0.2 -> 0.01
- board text added: "3V3"
- board text added: "<6.3V"
- board text added: "FEELER LEFT"
- board text added: "FEELER RIGHT"
- board text added: "GND"
- board text added: "IO"
- board text added: "L"
- board text added: "LINE LEFT IN"
- board text added: "LINE LEFT OUT"
- board text added: "LINE RIGHT IN"
- board text added: "LINE RIGHT OUT"
- board text added: "Minirobot 2016-02-23"
- board text added: "NRST"
- board text added: "PWR"
- board text added: "R"
- board text added: "RX"
- board text added: "SERVOS"
- board text added: "SIG VCC GND"
- board text added: "SWCLK"
- board text added: "SWDIO"
- board text added: "TX"
- board text added: "WHEEL LEFT"
- board text added: "WHEEL RIGHT"

Commit message: blink
Other:
- board text added: "4.3-6.3V"
- board text added: "ON"
- board text removed: "<6.3V"
Changed lines of the file:
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@@
-(kicad_pcb (version 4) (host pcbnew "(2016-01-20 BZR 6502, Git 4c1d9af)-product")
+(kicad_pcb (version 4) (host pcbnew "(2016-03-16 BZR 6623, Git 5de8545)-product")
   (general
     (links 171)
     (no_connects 0)
-    (area 97.650371 38.511799 180.978201 129.078201)
+    (area 97.725371 38.511799 180.978201 129.078201)
     (thickness 1.6)
-    (drawings 38)
+    (drawings 39)
     (tracks 826)
     (zones 0)
@@
       (hpglpenspeed 20)
       (hpglpendiameter 15)
-      (hpglpenoverlay 2)
       (psnegative false)
       (psa4output false)
@@
       (net 2 GNDPWR))
   )
+  (gr_text ON (at 118.4 93.4) (layer F.SilkS)
+    (effects (font (size 0.6 0.6) (thickness 0.1)) (justify left))
+  )
   (gr_text "SIG\nVCC\nGND" (at 106 92.7) (layer F.SilkS)
     (effects (font (size 0.4 0.4) (thickness 0.08)) (justify left))
@@
     (effects (font (size 0.6 0.6) (thickness 0.1)) (justify left))
   )
-  (gr_text <6.3V (at 108.2 93.5) (layer F.SilkS)
+  (gr_text 4.3-6.3V (at 108.2 93.5) (layer F.SilkS)
     (effects (font (size 0.6 0.6) (thickness 0.1)) (justify left))
   )
